File: STM32_SSD1306.kicad_sch (KiCad schematic)
At the start: 82 parts, among them J2 Conn_01x04_Pin, J2 USB_C_Receptacle_USB2.0, J3 Header_4P_2.54mm, J5 Conn_01x07_Pin, J8 Conn_01x04, Q1 2SC1815-HF, SW1 SW_Push, U2 ASM1117-3V3, U2 STM32F103C8Tx, U3 MAX485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

Commit message: Start Layout PCB
Parts:
- removed CT1: 100uF, Linktech:CP_Tantalum_Case-C_EIA-6032-28_Reflow, symbol ph_chemical_refrigerator_relay_hw-rescue:CT_6032-Linktech
- removed J2: Conn_01x04_Pin, symbol Connector:Conn_01x04_Pin
- added C19: 100nF, Capacitor_SMD:C_0805_2012Metric, symbol ph_kicad_lib:C0805
- added C20: 100nF, Capacitor_SMD:C_0805_2012Metric, symbol ph_chemical_refrigerator_relay_hw-rescue:C0805-ph_kicad_lib
- added C23: 10uF, Capacitor_SMD:C_0805_2012Metric, symbol ph_chemical_refrigerator_relay_hw-rescue:C0805-ph_kicad_lib
- added J6: Jack-DC, Connector_BarrelJack:BarrelJack_GCT_DCJ200-10-A_Horizontal, symbol Connector:Jack-DC
- added J7: Header_4P_2.54mm, Lib_Hien:Header_4P_2.54mm, symbol Lib_Hien:Header_4P_2.54mm
- added R22, R23: 4.7K, Resistor_SMD:R_0805_2012Metric, symbol Device:R
- C1, C11, C2, C20, C23: footprint ph_kicad_lib:C_0805_HandSoldering -> Capacitor_SMD:C_0805_2012Metric
- C18: footprint Linktech:C_1206_HandSoldering -> Capacitor_SMD:C_0805_2012Metric
- D7: footprint ph_kicad_lib:D_SMA -> Diode_SMD:D_SOD-128
- J2: footprint Connector_USB:USB_C_Receptacle_Palconn_UTC16-G -> Connector_USB:USB_C_Receptacle_GCT_USB4105-xx-A_16P_TopMnt_Horizontal
- J5: footprint (none) -> Connector_PinHeader_2.54mm:PinHeader_1x07_P2.54mm_Vertical
- J8: footprint ph_kicad_lib:Header-4pin-2.54 -> Connector_PinHeader_2.54mm:PinHeader_1x04_P2.54mm_Vertical
- L2: footprint ph_kicad_lib:L_0805_HandSoldering -> Inductor_SMD:L_0805_2012Metric
- R10, R11, R7, R8, R9: footprint ph_kicad_lib:R_0805_HandSoldering -> Resistor_SMD:R_0805_2012Metric
- U2: footprint Linktech:SOT-223 -> Package_TO_SOT_SMD:SOT-223
Connections:
- net +3.3V: now also R22.1, R23.1
- net +3V3: now also J8.2 (Pin_2), C19.2, C23.1, J7.2; no longer J8.1 (Pin_1)
- net +5V: now also C20.1
- net GND: now also J8.1 (Pin_1), C19.1, C20.2, C23.2, J6.2, J7.1; no longer J8.2 (Pin_2)
- net I2C1_SCL: now also U2.42 (PB6), J7.3, R23.2
- net I2C1_SDA: now also U2.43 (PB7), J7.4, R22.2
- net VCC renamed +12V
- net +12V: now also J6.1
Other:
- moved on the sheet: C11, C12, C13, C14, C18, C20, C23, D4, D5, D6, F3, L1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
